Commit message: adresses performance issues

File: urdf/test.xacro (robot description, xacro)
@@ -20,5 +20,5 @@
     <parent link="base_link" />
     <child link="base_sensor_link" />
-    <origin xyz="0 0 1.2" rpy="0 0 0" />
+    <origin xyz="0 0 4.2" rpy="0 0 0" />
   </joint>
   <joint name="imu_joint" type="fixed">
